File: hardware/ST_Link_V2.1.sch (KiCad schematic (older format))
At the start: 51 parts, among them J1 USB_C_Receptacle_USB2.0, J2 Conn_01x04, J3 Conn_03x05, Q1 Q_NPN_BEC, U1 STM32F103C8T6, U2 SPX3819M5-L-3-3, U3 AZ1117-3.3, Y1 SMD-5032_2P_8MHz_20ppm_20pF

Commit message: V1.0
Parts:
- removed J2: Conn_01x04, Connector_PinHeader_2.54mm:PinHeader_1x04_P2.54mm_Vertical, symbol Connector_Generic:Conn_01x04
- added J2: Conn_01x03, Connector_PinHeader_2.54mm:PinHeader_1x03_P2.54mm_Vertical, symbol Connector_Generic:Conn_01x03
Connections:
- net GND: now also J2.3 (Pin_3)
- net MCU_SWCLK: now also J2.2 (Pin_2)
- net MCU_SWDIO: now also J2.1 (Pin_1)
Changed lines of the file:
@@
-	1    0    0    -1
-$EndComp
-$Comp
-L Connector_Generic:Conn_01x04 J2
-U 1 1 60F84A64
-P 6200 3550
-F 0 "J2" H 6280 3542 50  0000 L CNN
-F 1 "Conn_01x04" H 6280 3451 50  0000 L CNN
-F 2 "Connector_PinHeader_2.54mm:PinHeader_1x04_P2.54mm_Vertical" H 6200 3550 50  0001 C CNN
-F 3 "~" H 6200 3550 50  0001 C CNN
-	1    6200 3550
 	1    0    0    -1
 $EndComp
@@
 Text Label 5600 3550 0    50   ~ 0
 MCU_SWDIO
-Wire Wire Line
-	5700 3450 6000 3450
-Wire Wire Line
-	5700 3250 5700 3450
-$Comp
-L power:+3.3V #PWR09
-U 1 1 60F86FFB
-P 5700 3250
-F 0 "#PWR09" H 5700 3100 50  0001 C CNN
-F 1 "+3.3V" H 5715 3423 50  0000 C CNN
-F 2 "" H 5700 3250 50  0001 C CNN
-F 3 "" H 5700 3250 50  0001 C CNN
-	1    5700 3250
-	1    0    0    -1
-$EndComp
 Wire Wire Line
 	9350 3650 9050 3650
@@
 $EndComp
 $Comp
-L power:+3.3V #PWR?
+L power:+3.3V #PWR0101
 U 1 1 614ED299
 P 10900 850
-F 0 "#PWR?" H 10900 700 50  0001 C CNN
+F 0 "#PWR0101" H 10900 700 50  0001 C CNN
 F 1 "+3.3V" H 10915 1023 50  0000 C CNN
 F 2 "" H 10900 850 50  0001 C CNN
@@
 Connection ~ 10900 900
 $Comp
-L power:+3.3VA #PWR?
+L power:+3.3VA #PWR0102
 U 1 1 614FBB55
 P 9050 3250
-F 0 "#PWR?" H 9050 3100 50  0001 C CNN
+F 0 "#PWR0102" H 9050 3100 50  0001 C CNN
 F 1 "+3.3VA" H 9065 3423 50  0000 C CNN
 F 2 "" H 9050 3250 50  0001 C CNN
@@
 $EndComp
 $Comp
-L power:+3.3VA #PWR?
+L power:+3.3VA #PWR0103
 U 1 1 614FC94B
 P 9750 3250
-F 0 "#PWR?" H 9750 3100 50  0001 C CNN
+F 0 "#PWR0103" H 9750 3100 50  0001 C CNN
 F 1 "+3.3VA" H 9765 3423 50  0000 C CNN
 F 2 "" H 9750 3250 50  0001 C CNN
@@
 $EndComp
 $Comp
-L power:+3.3VA #PWR?
+L power:+3.3VA #PWR0104
 U 1 1 614FCD93
 P 10450 3250
-F 0 "#PWR?" H 10450 3100 50  0001 C CNN
+F 0 "#PWR0104" H 10450 3100 50  0001 C CNN
 F 1 "+3.3VA" H 10465 3423 50  0000 C CNN
 F 2 "" H 10450 3250 50  0001 C CNN
@@
 $EndComp
 $Comp
-L power:+3.3VA #PWR?
+L power:+3.3VA #PWR0105
 U 1 1 614FD52E
 P 10650 2000
-F 0 "#PWR?" H 10650 1850 50  0001 C CNN
+F 0 "#PWR0105" H 10650 1850 50  0001 C CNN
 F 1 "+3.3VA" H 10665 2173 50  0000 C CNN
 F 2 "" H 10650 2000 50  0001 C CNN
@@
 Wire Wire Line
 	10650 2000 10650 2100
+$Comp
+L Connector_Generic:Conn_01x03 J2
+U 1 1 60EBA120
+P 6200 3650
+F 0 "J2" H 6280 3692 50  0000 L CNN
+F 1 "Conn_01x03" H 6280 3601 50  0000 L CNN
+F 2 "Connector_PinHeader_2.54mm:PinHeader_1x03_P2.54mm_Vertical" H 6200 3650 50  0001 C CNN
+F 3 "~" H 6200 3650 50  0001 C CNN
+	1    6200 3650
+	1    0    0    -1
+$EndComp
 $EndSCHEMATC
