File: hardware/ST_Link_V2.1.kicad_pcb (KiCad board)
At the start: 4 copper layers, 34.5 x 16 mm, 51 parts, among them J1 USB_C_Receptacle_USB2.0, J2 Conn_01x04, J3 Conn_03x05, Q1 Q_NPN_BEC, U1 STM32F103C8T6, U2 SPX3819M5-L-3-3, U3 AZ1117-3.3, Y1 SMD-5032_2P_8MHz_20ppm_20pF

Commit message: V1.0
Parts:
- J2: value Conn_01x04 -> Conn_01x03; footprint Connector_PinHeader_2.54mm:PinHeader_1x04_P2.54mm_Vertical -> Connector_PinHeader_2.54mm:PinHeader_1x03_P2.54mm_Vertical
- moved Y1 1.61 mm to (73.2, 87.4)
- moved J2 1.52 mm to (89.7, 81.5)
- moved JP1 1.25 mm to (79.5, 79.1)
Connections:
- C6 pad 2: GND -> Net-(F1-Pad2)
- J2 pad 1: +3V3 -> /MCU_SWDIO
- J2 pad 2: /MCU_SWDIO -> /MCU_SWCLK
- J2 pad 3: /MCU_SWCLK -> GND
Routing:
- net +5V: track 16.3 -> 46.9 mm
- net /MCU_SWCLK: track 0.00 -> 27.8 mm, vias 0 -> 1
- net +3V3: track 37.9 -> 63.3 mm, vias 2 -> 5
- net +3.3VA: track 20.4 -> 45.3 mm
- net /MCU_SWDIO: track 0.00 -> 24.6 mm, vias 0 -> 1
- net /SWCLK: track 0.00 -> 19.8 mm, vias 0 -> 2
- net /SWDIO: track 1.56 -> 19.4 mm, vias 0 -> 1
- net /SWIN: track 0.00 -> 14.4 mm, vias 0 -> 1
- net GND: track 1.42 -> 15.7 mm, vias 1 -> 6
- net Net-(F1-Pad2): track 0.00 -> 14.1 mm, vias 0 -> 1
- net /RESET: track 0.00 -> 11.3 mm, vias 0 -> 1
- net /MCU_USB_RENUM: track 0.00 -> 11.0 mm, vias 0 -> 2
- net /MCU_USB_D-: track 1.01 -> 11.9 mm, vias 1 -> 2
- net /BOOT0: track 0.00 -> 9.37 mm, vias 0 -> 2
- net /MCU_USB_D+: track 1.01 -> 9.58 mm, vias 1 -> 2
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
Commit message: 更改bug
Parts:
- removed JP1: SolderJumper_2_Bridged, Jumper:SolderJumper-2_P1.3mm_Bridged2Bar_Pad1.0x1.5mm
- D1, D2, D3, D4, D5: footprint LED_SMD:LED_0201_0603Metric -> LED_SMD:LED_0402_1005Metric
Connections:
- C6 pad 2: Net-(F1-Pad2) -> GND
- J1 pad A8: Net-(J1-PadA8) -> unconnected-(J1-PadA8)
- J1 pad B8: Net-(J1-PadB8) -> unconnected-(J1-PadB8)
- U1 pad 11: Net-(U1-Pad11) -> unconnected-(U1-Pad11)
- U1 pad 14: Net-(U1-Pad14) -> unconnected-(U1-Pad14)
- U1 pad 16: Net-(U1-Pad16) -> unconnected-(U1-Pad16)
- U1 pad 17: Net-(U1-Pad17) -> unconnected-(U1-Pad17)
- U1 pad 19: Net-(U1-Pad19) -> unconnected-(U1-Pad19)
- U1 pad 21: Net-(JP1-Pad1) -> GND
- U1 pad 22: Net-(U1-Pad22) -> unconnected-(U1-Pad22)
- U1 pad 28: Net-(U1-Pad28) -> unconnected-(U1-Pad28)
- U1 pad 29: Net-(U1-Pad29) -> unconnected-(U1-Pad29)
- U1 pad 39: Net-(U1-Pad39) -> unconnected-(U1-Pad39)
- U1 pad 4: Net-(U1-Pad4) -> unconnected-(U1-Pad4)
- U1 pad 40: Net-(U1-Pad40) -> unconnected-(U1-Pad40)
- U1 pad 41: Net-(U1-Pad41) -> unconnected-(U1-Pad41)
- U1 pad 42: Net-(U1-Pad42) -> unconnected-(U1-Pad42)
- U1 pad 43: Net-(U1-Pad43) -> unconnected-(U1-Pad43)
- U1 pad 45: Net-(U1-Pad45) -> unconnected-(U1-Pad45)
- U1 pad 46: Net-(U1-Pad46) -> unconnected-(U1-Pad46)
Routing:
- net Net-(JP1-Pad1): track 4.44 -> 0.00 mm
- net GND: track 15.7 -> 12.1 mm, vias 6 -> 7
- net Net-(Q1-Pad1): track 2.58 -> 4.47 mm
- net /TX: track 17.5 -> 16.7 mm
- net /SWIN: track 14.4 -> 15.1 mm
- net +3V3: track 63.3 -> 64.0 mm
Other:
- net class Default removed
